File: hw/k01/k01.brd (EAGLE design)
At the start: 160 x 100 mm, 1 part

Commit message: little updates
Parts:
- added U$1: RELAY-8-SRD, diy-modules:RELAY-8-SRD
- added U$2: MEGA_DEVICE, ArduinoMegaOutline:MEGAOUTLINE
- added U$3: DC-DC-STEP-DOWN-LM2596, diy-modules:DC-DC-STEP-DOWN-LM2596
Connections:
- new net GND.1: U$1.J1.10
- new net GND.2: U$1.J2.3
- new net VCC.1: U$1.J1.1
- new net VCC.2: U$1.J2.2
Changed lines of the file:
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@@
 <elements>
 <element name="D1" library="diode" library_urn="urn:adsk.eagle:library:210" package="DO35-10" package3d_urn="urn:adsk.eagle:package:43344/2" value="1N4148DO35-10" x="-25.4" y="38.1"/>
+<element name="U$1" library="diy-modules" package="RELAY-8-SRD" value="RELAY-8-SRD" x="-69.85" y="72.39"/>
+<element name="U$2" library="ArduinoMegaOutline" package="MEGAOUTLINE" value="MEGA_DEVICE" x="-46.99" y="-31.75"/>
+<element name="U$3" library="diy-modules" package="DC-DC-STEP-DOWN-LM2596" value="DC-DC-STEP-DOWN-LM2596" x="-64.77" y="-83.82"/>
 </elements>
 <signals>
+<signal name="VCC.1">
+<contactref element="U$1" pad="J1.1"/>
+</signal>
+<signal name="GND.1">
+<contactref element="U$1" pad="J1.10"/>
+</signal>
+<signal name="VCC.2">
+<contactref element="U$1" pad="J2.2"/>
+</signal>
+<signal name="GND.2">
+<contactref element="U$1" pad="J2.3"/>
+</signal>
 </signals>
 </board>

Commit message: little updates 2
Parts:
- removed D1: 1N4148DO35-10, diode:DO35-10
- moved U$3 183.5 mm to (12.7, 82.5), turned to 270 degrees
- moved U$2 172.5 mm to (77.5, 87.6)
- moved U$1 147.1 mm to (71.1, 30.5), turned to 90 degrees
Other:
- board size 160 x 100 mm -> 144.8 x 116.5 mm
Changed lines of the file:
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@@
 <board>
 <plain>
-<wire x1="0" y1="0" x2="160" y2="0" width="0" layer="20"/>
-<wire x1="160" y1="0" x2="160" y2="100" width="0" layer="20"/>
-<wire x1="160" y1="100" x2="0" y2="100" width="0" layer="20"/>
-<wire x1="0" y1="100" x2="0" y2="0" width="0" layer="20"/>
+<wire x1="0" y1="0" x2="143.49" y2="0" width="0" layer="20"/>
+<wire x1="143.49" y1="0" x2="143.49" y2="116.51" width="0" layer="20"/>
+<wire x1="143.49" y1="116.51" x2="-1.27" y2="116.51" width="0" layer="20"/>
+<wire x1="-1.27" y1="116.51" x2="0" y2="0" width="0" layer="20"/>
 </plain>
 <attributes>
@@
 </autorouter>
 <elements>
-<element name="D1" library="diode" library_urn="urn:adsk.eagle:library:210" package="DO35-10" package3d_urn="urn:adsk.eagle:package:43344/2" value="1N4148DO35-10" x="-25.4" y="38.1"/>
-<element name="U$1" library="diy-modules" package="RELAY-8-SRD" value="RELAY-8-SRD" x="-69.85" y="72.39"/>
-<element name="U$2" library="ArduinoMegaOutline" package="MEGAOUTLINE" value="MEGA_DEVICE" x="-46.99" y="-31.75"/>
-<element name="U$3" library="diy-modules" package="DC-DC-STEP-DOWN-LM2596" value="DC-DC-STEP-DOWN-LM2596" x="-64.77" y="-83.82"/>
+<element name="U$1" library="diy-modules" package="RELAY-8-SRD" value="RELAY-8-SRD" x="71.12" y="30.48" rot="R90"/>
+<element name="U$2" library="ArduinoMegaOutline" package="MEGAOUTLINE" value="MEGA_DEVICE" x="77.47" y="87.63"/>
+<element name="U$3" library="diy-modules" package="DC-DC-STEP-DOWN-LM2596" value="DC-DC-STEP-DOWN-LM2596" x="12.7" y="82.55" rot="R270"/>
 </elements>
 <signals>
@@
 </board>
 </drawing>
-<compatibility>
-<note version="8.2" severity="warning">
-Since Version 8.2, EAGLE supports online libraries. The ids
-of those online libraries will not be understood (or retained)
-with this version.
-</note>
-<note version="8.3" severity="warning">
-Since Version 8.3, EAGLE supports URNs for individual library
-assets (packages, symbols, and devices). The URNs of those assets
-will not be understood (or retained) with this version.
-</note>
-<note version="8.3" severity="warning">
-Since Version 8.3, EAGLE supports the association of 3D packages
-with devices in libraries, schematics, and board files. Those 3D
-packages will not be understood (or retained) with this version.
-</note>
-</compatibility>
 </eagle>
